File: kicad/revD/wsl-phase8b-revD.kicad_pcb (KiCad board)
At the start: 4 copper layers, 250 x 240 mm, 272 parts, among them J1 J_PI, J10 J_MOTION_M 5.08mm, J11 J_MOTION_M2 5.08mm, J12 J_MOTION_M1 5.08mm, J13 J_LAMP_LED, J14 J_SAFETY, J15 J_SLOW_IN_C, J16 J_EXT_I2C, J2 J_PWR 5V, J3 J_FAST_IN, J4 J_SLOW_IN_A, J5 J_SLOW_IN_B, J6 J_MOTION_S 5.08mm, J7 J_MOTION_T 5.08mm, J8 J_MOTION_SP 5.08mm, J9 J_MOTION_BE 5.08mm, K1 G5LE S, K2 G5LE T, K3 G5LE SP, K4 G5LE BE, K5 G5LE M, K6 G5LE M2, K7 G5LE M1 DNP, Q1 MMBT3904 S, Q10 2N7002 LED L_STRIKE, Q11 2N7002 LED L_FOUL, Q12 AO3400A kick, Q13 AO3400A wdog, Q14 AO3401A rail pass, Q15 MMBT3904 AND ARM, Q16 MMBT3904 AND RP_OK, Q2 MMBT3904 T, Q3 MMBT3904 SP, Q4 MMBT3904 BE, Q5 MMBT3904 M, Q6 MMBT3904 M2, Q7 MMBT3904 M1, Q8 2N7002 LED L_FIRST, Q9 2N7002 LED L_SECOND, U1 MCP23017 MCP_IN_A, U10 PC817 DIELL_L, U11 PC817 DIELL_R, U12 PC817 GS1, U13 PC817 GS2, U14 PC817 GS3, U15 PC817 GS4, U16 PC817 GS5, U17 PC817 GS6, U18 PC817 GS7, U19 PC817 GS8, U2 MCP23017 MCP_IN_B, U20 PC817 GS9, U21 PC817 GS10, U22 PC817 GP, U23 PC817 OS, U24 PC817 BS, U25 PC817 PBZ, U26 PC817 PBC, U27 PC817 FOUL, U28 PC817 TENTH, U29 PC817 MAN_T, U3 MCP23017 MCP_OUT_A, U30 PC817 MAN_S, U31 PC817 MAN_SWS, U32 PC817 MAN_SWSR, U33 PC817 AUX1, U34 PC817 AUX2, U35 PC817 AUX3, U36 PC817 AUX4, U37 PC817 AUX5, U38 PC817 AUX6, U39 PC817 AUX7, U4 PC817 SA, U40 PC817 AUX8, U41 PC817 AUX9, U42 PC817 AUX10, U43 PC817 AUX11, U44 NE555, U45 TMA-0505S, U5 PC817 SB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

Commit message: Phase 8 rev-D: board fully routed - DRC 0/0/0, routed-mode audit ALL PASS
New deterministic router (route_revD.py + lib + logic modules) in the rev-C
house style, re-derived for the rev-D placement; In1/In2 H/V discipline,
B.Cu backbones, logic-room-only GND zone, machine passes per rev-C pattern.
Built-in geometric self-check (0 problems). kicad-cli DRC: 0 violations,
0 unconnected, 0 footprint errors with live creepage rules; netclasses
re-applied before DRC; audit_revD_board.py (no --pre-route) ALL PASS.
Rev-C snapshot manifest verified 189/189 unchanged.

Co-Authored-By: Claude Fable 5 <noreply@anthropic.com>
Routing:
- net VCC_3V3: track 0.00 -> 772.9 mm, vias 0 -> 64
- net VCC_5V: track 0.00 -> 557.2 mm, vias 0 -> 16
- net RP2040_OK: track 0.00 -> 438.8 mm, vias 0 -> 11
- net FIELD_WET_V: track 0.00 -> 373.8 mm, vias 0 -> 43
- net FIELD_GND: track 0.00 -> 354.5 mm, vias 0 -> 4
- net I2C_SCL: track 0.00 -> 332.2 mm, vias 0 -> 10
- net RELAY_ENABLE_RAIL: track 0.00 -> 329.0 mm, vias 0 -> 9
- net GND: track 0.00 -> 299.4 mm, vias 0 -> 3
- net I2C_SDA: track 0.00 -> 299.4 mm, vias 0 -> 11
- net WDOG_TIMING_NODE: track 0.00 -> 279.0 mm, vias 0 -> 2
- net NE555_TRIG: track 0.00 -> 267.7 mm, vias 0 -> 4
- net NE555_OUT: track 0.00 -> 266.4 mm, vias 0 -> 5
- net SAFE_STOP_RETURN: track 0.00 -> 264.0 mm, vias 0 -> 3
- net ARM_PERMIT: track 0.00 -> 258.1 mm, vias 0 -> 4
- net WDOG_KICK: track 0.00 -> 239.6 mm, vias 0 -> 4
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- added copper zone on F.Cu, net GND

Commit message: Rev-D review-fix pass: power-via redundancy, honest gate records, HANDOFF update
- RD-VIA-1: doubled the five single-point power vias (VCC_5V x2,
  SAFE_STOP_RETURN x2, RELAY_ENABLE_RAIL spine entry) with parallel twin
  barrels + same-net stubs; copper-only. Post-fix gates: DRC 0/0/0
  (DRC-revD-routed-r3.rpt), netclasses 93/4/13/82/21, routed-mode audit
  ALL PASS, rev-C snapshot 189/189 unchanged.
- PV-1: routing was executed while blocking gate G8/OG-1 was open --
  recorded as a process violation, not sanctioned; routed artifact is
  conditional on Dylan's 240mm sign-off.
- Checklist G9/G10 updated to routed status (they contradicted the run
  log); first-article now gates on regenerated rev-D refdes test docs
  (46 REFDES_SHIFTs make every rev-C bench artifact wrong on rev-D).
- G8 enclosure re-check scope now includes row-39 bottom-edge copper
  (1.28mm to routed edge) alongside the COR-3 ribbon check.
- COR-4: external mirror predates routing -- routed board had no
  off-working-tree copy; new mirror WSL_Backups\2026-07-20_phase8_revD_routed.
- route_revD.py re-run instructions now pin the restore ref to e329872
  (1220c3e carries the divergent .kicad_pcb.bak hazard).
- HANDOFF.md: rev-D addendum (state, gates, REFDES_SHIFT trap, backups).

Co-Authored-By: Claude Fable 5 <noreply@anthropic.com>
Routing:
- net SAFE_STOP_RETURN: track 264.0 -> 267.9 mm, vias 3 -> 5
- net VCC_5V: track 557.2 -> 560.5 mm, vias 16 -> 18
- net RELAY_ENABLE_RAIL: track 329.0 -> 330.0 mm, vias 9 -> 10
Changed lines of the file:
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@@
+	)
+	(segment
+		(start 160 82)
+		(end 160 81)
+		(width 0.6)
+		(layer "F.Cu")
+		(net "RELAY_ENABLE_RAIL")
 	)
 	(segment
@@
 	(via
 		(at 160 82)
+		(size 0.8)
+		(drill 0.4)
+		(layers "F.Cu" "B.Cu")
+		(net "RELAY_ENABLE_RAIL")
+	)
+	(via
+		(at 160 81)
 		(size 0.8)
 		(drill 0.4)
@@
 	)
 	(segment
+		(start 118.4 20)
+		(end 118.4 21)
+		(width 0.5)
+		(layer "F.Cu")
+		(net "VCC_5V")
+	)
+	(segment
+		(start 167 14)
+		(end 164.7 14)
+		(width 0.5)
+		(layer "F.Cu")
+		(net "VCC_5V")
+	)
+	(segment
 		(start 167 10)
 		(end 167 14)
@@
 	)
 	(via
+		(at 164.7 14)
+		(size 0.8)
+		(drill 0.4)
+		(layers "F.Cu" "B.Cu")
+		(net "VCC_5V")
+	)
+	(via
 		(at 145.55 43.4)
 		(size 0.8)
@@
 	(via
 		(at 115.4 40)
+		(size 0.8)
+		(drill 0.4)
+		(layers "F.Cu" "B.Cu")
+		(net "VCC_5V")
+	)
+	(via
+		(at 118.4 21)
 		(size 0.8)
 		(drill 0.4)
@@
 	)
 	(segment
+		(start 177.5 13)
+		(end 176.5 13)
+		(width 0.6)
+		(layer "F.Cu")
+		(net "SAFE_STOP_RETURN")
+	)
+	(segment
 		(start 152.75 235.75)
 		(end 152 236)
@@
 	)
 	(via
+		(at 176.5 13)
+		(size 0.8)
+		(drill 0.4)
+		(layers "F.Cu" "B.Cu")
+		(net "SAFE_STOP_RETURN")
+	)
+	(via
 		(at 153.4 83.1)
 		(size 0.8)
@@
 	(via
 		(at 153.4 235.75)
+		(size 0.8)
+		(drill 0.4)
+		(layers "F.Cu" "B.Cu")
+		(net "SAFE_STOP_RETURN")
+	)
+	(via
+		(at 150.5 82.9228)
 		(size 0.8)
 		(drill 0.4)
@@
 		(width 0.6)
 		(layer "In1.Cu")
+		(net "SAFE_STOP_RETURN")
+	)
+	(segment
+		(start 153.4 83.1)
+		(end 150.5 82.9228)
+		(width 0.6)
+		(layer "In1.Cu")

Commit message: Rev-D board-chain remediation: R1 unidirectional taps + R2 rules/silk/drill, M2 router fix (Codex C1/H1/H2/M2/M3/M4)
- M2: route_revD --check-only reproducible on KiCad 10.0.2 (BOARD.Delete fix
  for the GetIsRuleArea crash/segfault after mass Remove); RD-VIA-1 twins now
  emitted by the router (route_power_via_redundancy) so the routed artifact
  regenerates from scripts alone.
- R1 (C1+H1): resistive taps replaced by four 2N7002 common-source stages
  (R_TAPIN 1M / R_TAPPU 10k / R_TAPG 10M; GPIO on drain only; inverted reads,
  fw v1.2 contract). 262 parts / 217 nets; netclasses 97/4/13/82/21 exact,
  Safety_Rail EXACTLY 13; ERC at the unchanged WVR-ERC-1 baseline (1+40);
  diff vs rev-C CLEAN, zero rev-C removals; 680k out, 1M/10M in. FR-8.
- R2 (H2): DRU re-derived from measured working voltages (FIELD <=14 V/34 Vpk
  basis; MACHINE <=37 Vpk) + IPC-2221B B1 + JLC +/-20% etch allowance ->
  2.65/3.35/1.6 mm; full re-route; kicad-cli DRC 0/0/0
  (DRC-revD-remediation-r3.rpt); routed-mode audit ALL PASS; measured minima
  L-F 2.650 / L-M 3.350 / ch-ch 2.325 mm.
- M3: F.SilkS floor 1.0 mm/0.15 enforced in add_text; KEYED warnings 1.2/0.20.
- M4: all 7 MCV connectors on project-local _D1.4 footprints (drill 1.4 mm,
  pad 2.0x3.6, annular 0.30 mm) in kicad/wsl_footprints.pretty; system lib
  untouched; VCC_3V3 trunk jogged around the widened J13.4 pad. FR-9.
- Docs: change spec E.2/E.3 superseded-marked + counts; change list
  remediation banner + item E rewrite (obsolete 3.27 V claim killed, M7);
  run log FR-8/FR-9 + board-chain record; readiness checklist G3/G4/G5/G9/G10
  refreshed; remediation spec committed.
- Rev-C sacred snapshot hash-verified 189/189 before and after.

Co-Authored-By: Claude Fable 5 <noreply@anthropic.com>
Parts:
- added Q17: 2N7002 TAP 555, Package_TO_SOT_SMD:SOT-23, F.Cu at (116.0, 52.0)
- added Q18: 2N7002 TAP KICK, Package_TO_SOT_SMD:SOT-23, F.Cu at (116.0, 56.0)
- added Q19: 2N7002 TAP ARM, Package_TO_SOT_SMD:SOT-23, F.Cu at (116.0, 60.0)
- added Q20: 2N7002 TAP RPOK, Package_TO_SOT_SMD:SOT-23, F.Cu at (116.0, 64.0)
- added R136: 1M, Resistor_SMD:R_0805_2012Metric, F.Cu at (130.0, 70.0)
- added R137: 10k, Resistor_SMD:R_0805_2012Metric, F.Cu at (120.5, 60.0)
- added R138: 10M, Resistor_SMD:R_0805_2012Metric, F.Cu at (125.0, 60.0)
- added R139: 1M, Resistor_SMD:R_0805_2012Metric, F.Cu at (156.0, 64.0)
- added R140: 10k, Resistor_SMD:R_0805_2012Metric, F.Cu at (120.5, 64.0)
- added R141: 10M, Resistor_SMD:R_0805_2012Metric, F.Cu at (125.0, 64.0)
- J13, J16: footprint Connector_Phoenix_MC:PhoenixContact_MCV_1,5_6-G-3.5_1x06_P3.50mm_Vertical -> wsl_footprints:PhoenixContact_MCV_1,5_6-G-3.5_1x06_P3.50mm_Vertical_D1.4
- J14: footprint Connector_Phoenix_MC:PhoenixContact_MCV_1,5_4-G-3.5_1x04_P3.50mm_Vertical -> wsl_footprints:PhoenixContact_MCV_1,5_4-G-3.5_1x04_P3.50mm_Vertical_D1.4
- J15, J3: footprint Connector_Phoenix_MC:PhoenixContact_MCV_1,5_10-G-3.5_1x10_P3.50mm_Vertical -> wsl_footprints:PhoenixContact_MCV_1,5_10-G-3.5_1x10_P3.50mm_Vertical_D1.4
- J4: footprint Connector_Phoenix_MC:PhoenixContact_MCV_1,5_14-G-3.5_1x14_P3.50mm_Vertical -> wsl_footprints:PhoenixContact_MCV_1,5_14-G-3.5_1x14_P3.50mm_Vertical_D1.4
- J5: footprint Connector_Phoenix_MC:PhoenixContact_MCV_1,5_12-G-3.5_1x12_P3.50mm_Vertical -> wsl_footprints:PhoenixContact_MCV_1,5_12-G-3.5_1x12_P3.50mm_Vertical_D1.4
- R131: value 100k -> 1M
- R132, R134: value 680k -> 10k
- R133: value 680k -> 1M
- R135: value 680k -> 10M
- moved R135 32.0 mm to (125.0, 56.0)
- moved R134 16.9 mm to (120.5, 56.0), turned to 180 degrees
- moved R132 14.0 mm to (120.5, 52.0), turned to 180 degrees
Connections:
- R131 pad 2: TAP_NE555_OUT -> TAP_GATE_555
- R132 pad 1: TAP_NE555_OUT -> VCC_3V3
- R132 pad 2: GND -> TAP_NE555_OUT
- R133 pad 2: TAP_WDOG_KICK -> TAP_GATE_KICK
- R134 pad 1: ARM_PERMIT -> VCC_3V3
- R134 pad 2: TAP_ARM_PERMIT -> TAP_WDOG_KICK
- R135 pad 1: RP2040_OK -> TAP_GATE_KICK
- R135 pad 2: TAP_RP2040_OK -> GND
Routing:
- net TAP_NE555_OUT: track 110.8 -> 16.0 mm
- net TAP_GATE_555: track 0.00 -> 61.6 mm, vias 0 -> 3
- net VCC_3V3: track 772.9 -> 818.7 mm, vias 64 -> 72
- net TAP_GATE_RPOK: track 0.00 -> 45.7 mm, vias 0 -> 2
- net TAP_RP2040_OK: track 72.3 -> 36.1 mm
- net TAP_GATE_KICK: track 0.00 -> 32.5 mm, vias 0 -> 3
- net TAP_ARM_PERMIT: track 53.9 -> 26.2 mm, vias 2 -> 3
- net TAP_WDOG_KICK: track 34.8 -> 12.3 mm, vias 2 -> 3
- net TAP_GATE_ARM: track 0.00 -> 22.5 mm, vias 0 -> 2
