File: kicad/revD/wsl-phase8b-revD.kicad_pcb (KiCad board)
At the start: 4 copper layers, 250 x 240 mm, 282 parts, among them J1 J_PI, J10 J_MOTION_M 5.08mm, J11 J_MOTION_M2 5.08mm, J12 J_MOTION_M1 5.08mm, J13 J_LAMP_LED, J14 J_SAFETY, J15 J_SLOW_IN_C, J16 J_EXT_I2C, J2 J_PWR 5V, J3 J_FAST_IN, J4 J_SLOW_IN_A, J5 J_SLOW_IN_B, J6 J_MOTION_S 5.08mm, J7 J_MOTION_T 5.08mm, J8 J_MOTION_SP 5.08mm, J9 J_MOTION_BE 5.08mm, K1 G5LE S, K2 G5LE T, K3 G5LE SP, K4 G5LE BE, K5 G5LE M, K6 G5LE M2, K7 G5LE M1 DNP, Q1 MMBT3904 S, Q10 2N7002 LED L_STRIKE, Q11 2N7002 LED L_FOUL, Q12 AO3400A kick, Q13 AO3400A wdog, Q14 AO3401A rail pass, Q15 MMBT3904 AND ARM, Q16 MMBT3904 AND RP_OK, Q17 2N7002 TAP 555, Q18 2N7002 TAP KICK, Q19 2N7002 TAP ARM, Q2 MMBT3904 T, Q20 2N7002 TAP RPOK, Q3 MMBT3904 SP, Q4 MMBT3904 BE, Q5 MMBT3904 M, Q6 MMBT3904 M2, Q7 MMBT3904 M1, Q8 2N7002 LED L_FIRST, Q9 2N7002 LED L_SECOND, U1 MCP23017 MCP_IN_A, U10 PC817 DIELL_L, U11 PC817 DIELL_R, U12 PC817 GS1, U13 PC817 GS2, U14 PC817 GS3, U15 PC817 GS4, U16 PC817 GS5, U17 PC817 GS6, U18 PC817 GS7, U19 PC817 GS8, U2 MCP23017 MCP_IN_B, U20 PC817 GS9, U21 PC817 GS10, U22 PC817 GP, U23 PC817 OS, U24 PC817 BS, U25 PC817 PBZ, U26 PC817 PBC, U27 PC817 FOUL, U28 PC817 TENTH, U29 PC817 MAN_T, U3 MCP23017 MCP_OUT_A, U30 PC817 MAN_S, U31 PC817 MAN_SWS, U32 PC817 MAN_SWSR, U33 PC817 AUX1, U34 PC817 AUX2, U35 PC817 AUX3, U36 PC817 AUX4, U37 PC817 AUX5, U38 PC817 AUX6, U39 PC817 AUX7, U4 PC817 SA, U40 PC817 AUX8, U41 PC817 AUX9, U42 PC817 AUX10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

Commit message: Round-2 board/BOM/export slice (Codex R2-2/R2-3/R2-4/R2-5/R2-6/R2-15)
- R2-4: J16 protection stack — 200mA polyfuse (Littelfuse 1206L020YR) on
  pin 1, default-OPEN solder link on pin 5, TCA4307 stuck-bus-recovery I2C
  buffer + 4.7k card-side pull-ups + bypass on pins 3/4, Semtech SRV05-4
  connector-side ESD array; J16 never touches a raw rail/bus (audit-enforced).
- R2-6: 2-bit REV_ID strap on GP20/GP21 (rev-D = 0b01; 0b00/floating =
  UNKNOWN); encoding recorded in run log + silk.
- R2-3: tap FETs Q17-Q20 MPN-locked to onsemi 2N7002LT1G (LCSC C16338) in
  value field + export hard lock (FR-10).
- R2-5: tap probe/fault-injection pads TP17-TP24 (gate+drain per stage, no
  SOT-23 pin probing) + fabricated TP silk legend + TP2 LOGIC GND / TP5
  FIELD GND / DO-NOT-BRIDGE marks.
- R2-2: retracted "~825k" R_TAPIN floor corrected to 1M (>=917k derated
  onset) in all 3 live spots; both repos swept.
- R2-15: exporter derives source paths from --rev (label defect dead), 10M
  pinned to LCSC C26108 (MATCH-AT-UPLOAD now export-fatal), coding-profile
  quantity corrected to 4/board (1 star + pilot spare).
- Board 262/217 -> 271/223, netclasses 103/4/13/82/21 (Safety_Rail 13
  unchanged); full re-route; DRC 0/0/0 (DRC-revD-round2-r4.rpt); routed
  audit ALL PASS; isolation minima unchanged 2.650/3.350 mm; diff vs rev-C
  CLEAN (zero removals); ERC baseline 1+39 (WVR-ERC-2).
- New as-ordered fab package kicad/fab_revD_2026-07-21_r2/ (271/28/243/226/
  26/17, sha256 manifest); first-article pack regenerated (271 rows, 24 TP).
- Run log: FR-10..FR-14, WVR-ERC-2, batch record; HANDOFF + checklist +
  remediation report supersession notes. rev-C snapshot 189/189 intact.

Co-Authored-By: Claude Fable 5 <noreply@anthropic.com>
Parts:
- added C16: 0.1uF, Capacitor_SMD:C_0805_2012Metric, F.Cu at (133.4, 216.4)
- added F1: 1206L020YR 200mA, Fuse:Fuse_1206_3216Metric, F.Cu at (122.6, 220.5)
- added JP1: 3V3 LINK OPEN DNP, Jumper:SolderJumper-2_P1.3mm_Open_RoundedPad1.0x1.5mm, F.Cu at (144.6, 218.9)
- added R142: 4.7k, Resistor_SMD:R_0805_2012Metric, F.Cu at (148.3, 216.0)
- added R143: 4.7k, Resistor_SMD:R_0805_2012Metric, F.Cu at (137.7, 223.3)
- added R144: 10k, Resistor_SMD:R_0805_2012Metric, F.Cu at (118.0, 68.0)
- added R145: 10k, Resistor_SMD:R_0805_2012Metric, F.Cu at (118.0, 71.0)
- added TP17: TAP_GATE_555, TestPoint:TestPoint_Pad_1.0x1.0mm, F.Cu at (128.0, 53.8)
- added TP18: TAP_NE555_OUT, TestPoint:TestPoint_Pad_1.0x1.0mm, F.Cu at (112.8, 52.0)
- added TP19: TAP_GATE_KICK, TestPoint:TestPoint_Pad_1.0x1.0mm, F.Cu at (128.0, 57.8)
- added TP20: TAP_WDOG_KICK, TestPoint:TestPoint_Pad_1.0x1.0mm, F.Cu at (112.8, 56.0)
- added TP21: TAP_GATE_ARM, TestPoint:TestPoint_Pad_1.0x1.0mm, F.Cu at (128.0, 61.8)
- added TP22: TAP_ARM_PERMIT, TestPoint:TestPoint_Pad_1.0x1.0mm, F.Cu at (112.8, 60.0)
- added TP23: TAP_GATE_RPOK, TestPoint:TestPoint_Pad_1.0x1.0mm, F.Cu at (128.0, 65.8)
- added TP24: TAP_RP2040_OK, TestPoint:TestPoint_Pad_1.0x1.0mm, F.Cu at (112.8, 64.0)
- added U46: TCA4307DGKR, Package_SO:VSSOP-8_3x3mm_P0.65mm, F.Cu at (130.9, 220.6)
- added U47: SRV05-4, Package_TO_SOT_SMD:SOT-23-6, F.Cu at (140.3, 217.2)
- Q17: value 2N7002 TAP 555 -> 2N7002LT1G TAP 555
- Q18: value 2N7002 TAP KICK -> 2N7002LT1G TAP KICK
- Q19: value 2N7002 TAP ARM -> 2N7002LT1G TAP ARM
- Q20: value 2N7002 TAP RPOK -> 2N7002LT1G TAP RPOK
Connections:
- A1 pad 26: (no net) -> REV_ID0
- A1 pad 27: (no net) -> REV_ID1
- J16 pad 1: VCC_5V -> J16_5V
- J16 pad 3: I2C_SDA -> J16_SDA
- J16 pad 4: I2C_SCL -> J16_SCL
- J16 pad 5: VCC_3V3 -> J16_3V3
Routing:
- net VCC_3V3: track 818.7 -> 872.4 mm, vias 72 -> 78
- net I2C_SDA: track 299.4 -> 344.6 mm, vias 11 -> 14
- net REV_ID1: track 0.00 -> 37.9 mm, vias 0 -> 3
- net J16_5V: track 0.00 -> 35.8 mm, vias 0 -> 4
- net REV_ID0: track 0.00 -> 34.0 mm, vias 0 -> 3
- net J16_SCL: track 0.00 -> 32.6 mm, vias 0 -> 2
- net J16_SDA: track 0.00 -> 29.1 mm, vias 0 -> 3
- net VCC_5V: track 560.5 -> 534.5 mm
- net J16_3V3: track 0.00 -> 16.4 mm
- net I2C_SCL: track 332.2 -> 319.1 mm, vias 10 -> 8
- net TAP_GATE_555: track 61.6 -> 64.4 mm
- net TAP_GATE_RPOK: track 45.7 -> 47.8 mm
- net TAP_GATE_KICK: track 32.5 -> 34.6 mm
- net TAP_GATE_ARM: track 22.5 -> 23.9 mm
- net TAP_WDOG_KICK: track 12.3 -> 13.6 mm
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Other:
- board text added: "D"
- board text added: "DO NOT BRIDGE TO TP2"
- board text added: "DO NOT BRIDGE TO TP5"
- board text added: "G"
- board text added: "REV ID D=01"
- board text added: "TAP PROBES: D WEST / G EAST"
- board text added: "TP1 5V"
- board text added: "TP10 TRG"
- board text added: "TP11 555"
- board text added: "TP12 WOK"
- board text added: "TP13 ARM"
- board text added: "TP14 RPO"
- board text added: "TP15 SAFE"
- board text added: "TP16 RAIL"
- board text added: "TP2 LOGIC GND"
- board text added: "TP3 3V3"
- board text added: "TP4 WET V"
- board text added: "TP5 FIELD GND"
- board text added: "TP6 SDA"
- board text added: "TP7 SCL"
- board text added: "TP8 KICK"
- board text added: "TP9 TMG"
